File: projects/ucontroller/uController_hub.sch (KiCad schematic (older format))
At the start: 1 part

Commit message: Fix symbol and footprint libraries
Parts:
- U?: symbol PIC24:PIC24FV32KA301 -> OARS:PIC24FV32KA301
Changed lines of the file:
@@
 EESchema Schematic File Version 4
+LIBS:uController_hub-cache
 EELAYER 26 0
 EELAYER END
@@
 $EndDescr
 $Comp
-L PIC24:PIC24FV32KA301 U?
+L OARS:PIC24FV32KA301 U?
 U 1 1 5C66DFEB
 P 5800 3850

Commit message: uController Hub First Draft
Brings USB hub, Power Adapter, and uController subcircuits together into one
TODO: Add battery connector, windvane connector, check buck converters, and investigate using Jetson to supply 3.3V
Parts:
- added C1, C17, C28, C29, C4, C5, C8: 150uF, symbol Device:CP1
- added C10, C11, C13, C14, C16, C22, C23, C25, C26, C33, C34, C35, C36, C38, C39, C40, C41, C7: 0.1uF, symbol OARS:C
- added C12, C24, C32, C44: 100uF, symbol OARS:C
- added C15, C27, C3, C37: 100uF, symbol Device:CP1
- added C18, C19: 6pF, symbol OARS:C
- added C2: 1nF, symbol OARS:C
- added C20, C30, C42, C6: 470pF, symbol OARS:C
- added C21, C31, C43, C9: 470uF, symbol Device:CP1
- added C45, C47: 100nF, symbol OARS:C
- added C46, C51: 100 nF, symbol OARS:C
- added C48: 6.8nF, symbol OARS:C
- added C49: 120nF, symbol OARS:C
- added C50: 10 uF, symbol OARS:C
- added D1, D2, D3, D4: D_Zener, symbol Device:D_Zener
- added J1, J2, J4: USB_A, symbol OARS:USB_A
- added J10: SERVO_CONN, symbol Connector_Generic:Conn_01x04
- added J11: Conn_02x20_Odd_Even, symbol Connector_Generic:Conn_02x20_Odd_Even
- added J3, J5, J6, J7, J8: USB3_A, symbol OARS:USB3_A
- added J9: PICKIT_CONN, symbol Connector_Generic:Conn_01x05
- added L1, L3, L5, L7: 220uH, symbol Device:L_Core_Iron
- added L2, L4, L6, L8: 1uH, symbol Device:L_Core_Iron
- added R1, R10, R17, R6: 0.33, symbol OARS:R
- added R11, R2, R23, R7: 1.2k, symbol OARS:R
- added R12: 2k, symbol OARS:R
- added R13, R14, R15, R16, R19, R20, R21, R22: 330, symbol OARS:R
- added R18: 30k, symbol OARS:R
- added R24, R25, R26, R27, R28: 10k, symbol Device:R
- added R29: 470, symbol Device:R
- added R3, R4: 100k, symbol OARS:R
- added R5: 10k, symbol OARS:R
- added R8: 12k, symbol OARS:R
- added R9: 3.6k, symbol OARS:R
- added SW1: PIC_RESET, symbol Switch:SW_Push
- added U1, U3, U4, U5: AZ34063U, symbol OARS:AZ34063U
- added U2: USB5537B, symbol OARS:USB5537B
- added U6: IMU(BNO055), Package_LGA:LGA-28_5.2x3.8mm_P0.5mm, symbol Sensor_Motion:BNO055
- added Y1: XTAL_GND, symbol OARS:XTAL_GND
- U7: renamed from U?; symbol OARS:PIC24FV32KA301 -> uController_hub-rescue:PIC24FV32KA301-OARS
Connections:
- net MCLR: now reaches U7.1 (MCLR/RA5)
- net MCLR: now also J9.1 (Pin_1), R29.1
- net OC1: now reaches U7.11 (RB7)
- net OC1: now also J10.1 (Pin_1)
- net at U7.14 (RA6/VCAP): now also C50.1
- net SCK1: now reaches U7.15 (RB12)
- net SCK1: now also J11.23 (Pin_23)
- net SDO1: now reaches U7.16 (RB13)
- net SDO1: now also J11.21 (Pin_21)
- net SDI1: now reaches U7.17 (RB14)
- net SDI1: now also J11.19 (Pin_19)
- net SS1: now reaches U7.18 (RB15)
- net SS1: now also J11.24 (Pin_24)
- net GND: now reaches U7.19 (VSS)
- net GND: now also C1.2, C12.2, C17.2, C18.1, C19.1, C2.2, C20.2, C21.2, C24.2, C28.2, C29.2, C30.2, C31.2, C32.2, C33.1, C33.2, C34.1, C34.2, C35.1, C35.2, C36.1, C36.2, C38.1, C38.2, C39.1, C39.2, C4.2, C40.1, C40.2, C41.1, C41.2, C42.2, C43.2, C44.2, C45.2, C46.2, C47.2, C48.2, C49.2, C5.2, C50.2, C51.2, C6.2, C8.2, C9.2, D1.2 (A), D2.2 (A), D3.2 (A), D4.2 (A), J1.4 (GND), J1.5 (Shield), J10.4 (Pin_4), J11.14 (Pin_14), J11.20 (Pin_20), J11.25 (Pin_25), J11.30 (Pin_30), J11.34 (Pin_34), J11.39 (Pin_39), J11.6 (Pin_6), J11.9 (Pin_9), J2.4 (GND), J2.5 (Shield), J3.10 (SHIELD), J3.4 (GND), J3.7 (DRAIN), J4.4 (GND), J4.5 (Shield), J5.10 (SHIELD), J5.4 (GND), J5.7 (DRAIN), J6.10 (SHIELD), J6.4 (GND), J6.7 (DRAIN), J7.10 (SHIELD), J7.4 (GND), J7.7 (DRAIN), J8.10 (SHIELD), J8.4 (GND), J8.7 (DRAIN), J9.3 (Pin_3), R11.1, R13.1, R13.2, R14.1, R14.2, R15.1, R15.2, R16.1, R16.2, R18.1, R19.1, R19.2, R2.1, R20.1, R20.2, R21.1, R21.2, R22.1, R22.2, R4.1, R7.1, R8.1, SW1.1, U1.4 (GND), U2.68 (ATEST), U3.4 (GND), U4.4 (GND), U5.4 (GND), U6.10 (BL_IND), U6.15 (GNDIO), U6.16 (GNDIO), U6.17 (COM3), U6.18 (COM2), U6.2 (GND), U6.25 (GNDIO), U6.5 (PS1), U6.6 (PS0), Y1.3
- net PGEC: now reaches U7.2 (RA0)
- net PGEC: now also J9.5 (Pin_5)
- net +5V: now reaches U7.20 (VDD)
- net +5V: now also C24.1, C51.1, J9.2 (Pin_2), L4.2, R28.1
- net PGED: now reaches U7.3 (RA1)
- net PGED: now also J9.4 (Pin_4)
- net OC2: now reaches U7.4 (RB0)
- net OC2: now also J10.2 (Pin_2)
- net OC3: now reaches U7.5 (RB1)
- net OC3: now also J10.3 (Pin_3)
- new net: J7.3 (D+), U2.11 (USB2DP_DN2)
- new net: J7.2 (D-), U2.12 (USB2DM_DN2)
- new net: C25.2, U2.13 (USB3DP_TXDN2)
- new net: C22.2, U2.14 (USB3DM_TXDN2)
- new net: J7.6 (SSRX+), U2.16 (USB3DP_RXDN2)
- new net: J7.5 (SSRX-), U2.17 (USB3DM_RXDN2)
- new net: J5.3 (D+), U2.19 (USB2DP_DN3)
- new net: J5.2 (D-), U2.20 (USB2DM_DN3)
- new net: C16.2, U2.21 (USB3DP_TXDN3)
- new net: C14.2, U2.22 (USB3DM_TXDN3)
- new net: J5.6 (SSRX+), U2.24 (USB3DP_RXDN3)
- new net: J5.5 (SSRX-), U2.25 (USB3DM_RXDN3)
- new net: J3.3 (D+), U2.26 (USB2DP_DN4)
- new net: J3.2 (D-), U2.27 (USB2DM_DN4)
- new net: C7.2, U2.28 (USB3DP_TXDN4)
- new net: C10.2, U2.29 (USB3DM_TXDN4)
- new net: J8.3 (D+), U2.3 (USB2DP_DN1)
- new net: J3.6 (SSRX+), U2.31 (USB3DP_RXDN4)
- new net: J3.5 (SSRX-), U2.32 (USB3DM_RXDN4)
- new net: J1.3 (D+), U2.33 (USB2DP_DN5)
- new net: J1.2 (D-), U2.34 (USB2DM_DN5)
- new net: J8.2 (D-), U2.4 (USB2DM_DN1)
- new net: C26.2, U2.5 (USB3DP_TXDN1)
- new net: R3.1, R4.2, U2.52 (VBUS)
- new net: J2.2 (D-), U2.57 (USB2DM_DN6)
- new net: J2.3 (D+), U2.58 (USB2DP_DN6)
- new net: J4.2 (D-), U2.59 (USB2DM_DN7)
- new net: C23.2, U2.6 (USB3DM_TXDN1)
- new net: J4.3 (D+), U2.60 (USB2DP_DN7)
- new net: J6.3 (D+), U2.61 (USB2DP_UP)
- new net: J6.2 (D-), U2.62 (USB2DM_UP)
- new net: C11.1, U2.63 (USB3DP_TXUP)
- new net: C13.1, U2.64 (USB3DM_TXUP)
- new net: J6.6 (SSRX+), U2.66 (USB3DP_RXUP)
- new net: J6.5 (SSRX-), U2.67 (USB3DM_RXUP)
- new net: C19.2, U2.69 (XTALOUT), Y1.1
- new net: C18.2, U2.70 (XTALIN), Y1.2
- new net: R8.2, U2.72 (RBIAS)
- new net: J8.6 (SSRX+), U2.8 (USB3DP_RXDN1)
- new net: J8.5 (SSRX-), U2.9 (USB3DM_RXDN1)
- new net: C23.1, J8.8 (SSTX-)
- new net: C26.1, J8.9 (SSTX+)
- new net: C22.1, J7.8 (SSTX-)
- new net: C25.1, J7.9 (SSTX+)
- new net: C14.1, J5.8 (SSTX-)
- new net: C16.1, J5.9 (SSTX+)
- new net: C10.1, J3.8 (SSTX-)
- new net: C7.1, J3.9 (SSTX+)
- new net: C9.1, L1.2, L2.1, R5.1
- new net: R1.1, U1.1 (S_COL), U1.7 (IPK_SENSE), U1.8 (DRV_COL)
- new net: D1.1 (K), L1.1, U1.2 (S_EMT)
- new net: C6.1, U1.3 (TMG_CAP)
- new net: C3.2, R2.2, R5.2, U1.5 (CI_INPUT)
- new net: C13.2, J6.8 (SSTX-)
- new net: C11.2, J6.9 (SSTX+)
- new net: C21.1, L3.2, L4.1, R9.1
- new net: R6.1, U3.1 (S_COL), U3.7 (IPK_SENSE), U3.8 (DRV_COL)
- new net: D2.1 (K), L3.1, U3.2 (S_EMT)
- new net: C20.1, U3.3 (TMG_CAP)
- new net: C15.2, R7.2, R9.2, U3.5 (CI_INPUT)
- new net: C46.1, R28.2, R29.2, SW1.2
- new net: R27.2, U6.11 (~nRESET)
- new net: R26.2, U6.4 (~nBOOT_LOAD_PIN)
- new net: C47.1, U6.9 (CAP)
- new net: C31.1, L5.2, L6.1, R12.1
- new net: R10.1, U4.1 (S_COL), U4.7 (IPK_SENSE), U4.8 (DRV_COL)
- new net: D3.1 (K), L5.1, U4.2 (S_EMT)
- new net: C30.1, U4.3 (TMG_CAP)
- new net: C27.2, R11.2, R12.2, U4.5 (CI_INPUT)
- new net: C43.1, L7.2, L8.1, R23.1
- new net: R17.1, U5.1 (S_COL), U5.7 (IPK_SENSE), U5.8 (DRV_COL)
- new net: D4.1 (K), L7.1, U5.2 (S_EMT)
- new net: C42.1, U5.3 (TMG_CAP)
- new net: C37.2, R18.2, R23.2, U5.5 (CI_INPUT)
- new net +12V: C12.1, L2.2
- new net +1V2: C44.1, L8.2, U2.10 (VDD12), U2.15 (VDD12), U2.23 (VDD12), U2.30 (VDD12), U2.35 (VDD12), U2.55 (VDD12), U2.65 (VDD12), U2.7 (VDD12)
- new net +3V3: C32.1, C45.1, C48.1, C49.1, L6.2, R24.1, R25.1, R26.1, R27.1, U2.18 (VDD33), U2.56 (VDD33), U2.71 (VDD33), U6.28 (VDDIO), U6.3 (VDD)
- new net 5V_PRT1: C29.1, J8.1 (VBUS), U2.39 (PRT_PWR1)
- new net 5V_PRT2: C28.1, J7.1 (VBUS), U2.38 (PRT_PWR2)
- new net 5V_PRT3: C17.1, J5.1 (VBUS), U2.37 (PRT_PWR3)
- new net 5V_PRT4: C8.1, J3.1 (VBUS), U2.36 (PRT_PWR4)
- new net 5V_PRT5: C1.1, J1.1 (VBUS), U2.40 (PRT_PWR5)
- new net 5V_PRT6: C4.1, J2.1 (VBUS), U2.2 (PRT_PWR6)
- new net 5V_PRT7: C5.1, J4.1 (VBUS), U2.1 (PRT_PWR7)
- new net M_INT: J11.31 (Pin_31), U6.14 (INT)
- new net SCL: J11.5 (Pin_5), R24.2, U6.19 (COM1)
- new net SDA: J11.3 (Pin_3), R25.2, U6.20 (COM0)
- new net VBUS: C2.1, J6.1 (VBUS), R3.2
- new net VCC: C15.1, C27.1, C3.1, C37.1, R1.2, R10.2, R17.2, R6.2, U1.6 (VCC), U3.6 (VCC), U4.6 (VCC), U5.6 (VCC)
- no-connect marks 0 -> 13
Other:
- note added: "1: MCLR, Master Clear\n2: PGEC, Programmer Communication \n3: PGED, Programmer Communication \n4: OC2, PWM for servo #2\n5: OC3, PWM for servo #3\n11: OC1, PWM for servo #1\n14: VCAP, see PIC datasheet\n15: SCK1, SPI Clock\n16: SDO1, SPI Data Out\n17: SDI1, SPI Data In\n18: SS1, Slave Select1 (input)\n19: VSS, Ground\n20: VDD, +5V Supply"
- note added: "IMU (Motion Sensor)\nConnected directly to Jetson\nI2C Addr.: 0x28"
- note added: "PICKIT3 Connector\nfor Programming"
- note added: "SPI Connection:\nPIC operates as Slave\nSDI1 is Master Out/Slave In\nSDO1 is Master In/Slave out\nSS1 is Active-Low Slave Select"
- note added: "Servo Control Connector\nSignals Only, No Power\nOC1, OC2, & OC3 are PWM"

Commit message: Update uController
Parts:
- removed C1, C17, C28, C29, C4, C5, C8: 150uF, symbol Device:CP1
- removed C10, C11, C13, C14, C16, C22, C23, C25, C26, C33, C34, C35, C36, C38, C39, C40, C41, C7: 0.1uF, symbol OARS:C
- removed C12, C24, C32, C44: 100uF, symbol OARS:C
- removed C15, C27, C3, C37: 100uF, symbol Device:CP1
- removed C18, C19: 6pF, symbol OARS:C
- removed C2: 1nF, symbol OARS:C
- removed C20, C30, C42, C6: 470pF, symbol OARS:C
- removed C21, C31, C43, C9: 470uF, symbol Device:CP1
- removed D1, D2, D3, D4: D_Zener, symbol Device:D_Zener
- removed J1, J2, J4: USB_A, symbol OARS:USB_A
- removed J3, J5, J6, J7, J8: USB3_A, symbol OARS:USB3_A
- removed L1, L3, L5, L7: 220uH, symbol Device:L_Core_Iron
- removed L2, L4, L6, L8: 1uH, symbol Device:L_Core_Iron
- removed R1, R10, R17, R6: 0.33, symbol OARS:R
- removed R11, R2, R23, R7: 1.2k, symbol OARS:R
- removed R12: 2k, symbol OARS:R
- removed R13, R14, R15, R16, R19, R20, R21, R22: 330, symbol OARS:R
- removed R18: 30k, symbol OARS:R
- removed R3, R4: 100k, symbol OARS:R
- removed R5: 10k, symbol OARS:R
- removed R8: 12k, symbol OARS:R
- removed R9: 3.6k, symbol OARS:R
- removed U1, U3, U4, U5: AZ34063U, symbol OARS:AZ34063U
- removed U2: USB5537B, symbol OARS:USB5537B
- removed Y1: XTAL_GND, symbol OARS:XTAL_GND
- J3: renamed from J11; value Conn_02x20_Odd_Even -> JETSON_TX2_CONN
- renumbered C45 to C1, C46 to C2, C47 to C3, C48 to C4, C49 to C5, C50 to C6, C51 to C7, J9 to J1, J10 to J2, R24 to R1, R25 to R2, R26 to R3, R27 to R4, R28 to R5, R29 to R6, U6 to U1, U7 to U2
Connections:
- no-connect marks 13 -> 0
Other:
- moved on the sheet: C1, C2, C3, C4, C5, C6, C7, J1, J2, J3, R1, R2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

Commit message: Update uController
Parts:
- removed J2: SERVO_CONN, symbol Connector_Generic:Conn_01x04
- added J3: SERVO1, symbol Connector_Generic:Conn_01x03
- added J4: SERVO2, symbol Connector_Generic:Conn_01x03
- added J5: SERVO3, symbol Connector_Generic:Conn_01x03
- U2: symbol uController_hub-rescue:PIC24FV32KA301-OARS -> OARS:PIC24FV32KA301
- renumbered C4 to C2, C5 to C3, C3 to C4, C7 to C5, C2 to C6, C6 to C7, J3 to J1, J1 to J2
Connections:
- net GND: now also J3.3 (Pin_3), J4.3 (Pin_3), J5.3 (Pin_3)
- net OC1: now also J3.1 (Pin_1)
- net OC2: now also J4.1 (Pin_1)
- net OC3: now also J5.1 (Pin_1)
- new net +12V: J3.2 (Pin_2), J4.2 (Pin_2), J5.2 (Pin_2)
Other:
- note added: "Designer: Michael Remley"
- note added: "Servo Control Connector\nSignals and 12V Power\nOC1, OC2, & OC3 are 5V PWM"
- note added: "uController"
- note removed: "Servo Control Connector\nSignals Only, No Power\nOC1, OC2, & OC3 are PWM"

Commit message: uController Circuit Footprints Added
Parts:
- C1, C2, C3, C4, C5, C6, C7: footprint (none) -> Capacitor_SMD:C_0603_1608Metric_Pad1.05x0.95mm_HandSolder
- J1: footprint (none) -> Connector_PinHeader_2.54mm:PinHeader_2x20_P2.54mm_Vertical
- J2: footprint (none) -> Connector_PinHeader_2.54mm:PinHeader_1x05_P2.54mm_Horizontal
- J3, J4, J5: footprint (none) -> Connector_PinHeader_2.54mm:PinHeader_1x03_P2.54mm_Vertical
- R1, R2, R3, R4, R5, R6: footprint (none) -> Resistor_SMD:R_0603_1608Metric_Pad1.05x0.95mm_HandSolder
- U2: footprint (none) -> OARS:PIC24FV32KA301-SOIC
Connections:
- net MCLR: now also C6.1, R5.2, R6.2, SW1.2; no longer R6.1, U2.1 (MCLR/RA5)
- new net: R6.1, U2.1 (MCLR/RA5)
Changed lines of the file:
@@
 EESchema Schematic File Version 4
 LIBS:uController_hub-cache
-LIBS:power_adapter-cache
-LIBS:usb-cache
 EELAYER 26 0
 EELAYER END
@@
 F 0 "U2" V 4965 4500 50  0000 C CNN
 F 1 "PIC24FV32KA301" V 4874 4500 50  0000 C CNN
-F 2 "" H 4250 4450 50  0001 C CNN
+F 2 "OARS:PIC24FV32KA301-SOIC" H 4250 4450 50  0001 C CNN
 F 3 "" H 4250 4450 50  0001 C CNN
 	1    4250 4450
@@
 F 0 "C6" H 3115 4196 50  0000 L CNN
 F 1 "100 nF" H 3115 4105 50  0000 L CNN
-F 2 "" H 3038 4000 50  0001 C CNN
+F 2 "Capacitor_SMD:C_0603_1608Metric_Pad1.05x0.95mm_HandSolder" H 3038 4000 50  0001 C CNN
 F 3 "" H 3000 4150 50  0001 C CNN
 	1    3000 4150
@@
 F 0 "C5" H 5715 4046 50  0000 L CNN
 F 1 "100 nF" H 5715 3955 50  0000 L CNN
-F 2 "" H 5638 3850 50  0001 C CNN
+F 2 "Capacitor_SMD:C_0603_1608Metric_Pad1.05x0.95mm_HandSolder" H 5638 3850 50  0001 C CNN
 F 3 "" H 5600 4000 50  0001 C CNN
 	1    5600 4000
@@
 F 0 "C7" H 5565 4796 50  0000 L CNN
 F 1 "10 uF" H 5565 4705 50  0000 L CNN
-F 2 "" H 5488 4600 50  0001 C CNN
+F 2 "Capacitor_SMD:C_0603_1608Metric_Pad1.05x0.95mm_HandSolder" H 5488 4600 50  0001 C CNN
 F 3 "" H 5450 4750 50  0001 C CNN
 	1    5450 4750
@@
 F 0 "R6" V 2993 4000 50  0000 C CNN
 F 1 "470" V 3084 4000 50  0000 C CNN
-F 2 "" V 3130 4000 50  0001 C CNN
+F 2 "Resistor_SMD:R_0603_1608Metric_Pad1.05x0.95mm_HandSolder" V 3130 4000 50  0001 C CNN
 F 3 "" H 3200 4000 50  0001 C CNN
 	1    3200 4000
@@
 F 0 "R5" H 2930 3696 50  0000 R CNN
 F 1 "10k" H 2930 3605 50  0000 R CNN
-F 2 "" V 2930 3650 50  0001 C CNN
+F 2 "Resistor_SMD:R_0603_1608Metric_Pad1.05x0.95mm_HandSolder" V 2930 3650 50  0001 C CNN
 F 3 "" H 3000 3650 50  0001 C CNN
 	1    3000 3650
@@
 	3000 4000 3050 4000
 Wire Wire Line
-	3000 4000 3000 3800
+	3000 4000 3000 3900
 Connection ~ 3000 4000
-Wire Wire Line
-	3350 4000 3650 4000
 $Comp
 L Switch:SW_Push SW1
@@
 F 0 "J2" H 1370 4517 50  0000 C CNN
 F 1 "PICKIT_CONN" H 1370 4426 50  0000 C CNN
-F 2 "" H 1450 4100 50  0001 C CNN
+F 2 "Connector_PinHeader_2.54mm:PinHeader_1x05_P2.54mm_Horizontal" H 1450 4100 50  0001 C CNN
 F 3 "" H 1450 4100 50  0001 C CNN
 	1    1450 4100
@@
 F 0 "C4" H 3815 2496 50  0000 L CNN
 F 1 "100nF" H 3815 2405 50  0000 L CNN
-F 2 "" H 3738 2300 50  0001 C CNN
+F 2 "Capacitor_SMD:C_0603_1608Metric_Pad1.05x0.95mm_HandSolder" H 3738 2300 50  0001 C CNN
 F 3 "" H 3700 2450 50  0001 C CNN
 	1    3700 2450
@@
 F 0 "C1" H 1815 1296 50  0000 L CNN
 F 1 "100nF" H 1815 1205 50  0000 L CNN
-F 2 "" H 1738 1100 50  0001 C CNN
+F 2 "Capacitor_SMD:C_0603_1608Metric_Pad1.05x0.95mm_HandSolder" H 1738 1100 50  0001 C CNN
 F 3 "" H 1700 1250 50  0001 C CNN
 	1    1700 1250
@@
 F 0 "C2" H 3865 1296 50  0000 L CNN
 F 1 "6.8nF" H 3865 1205 50  0000 L CNN
-F 2 "" H 3788 1100 50  0001 C CNN
+F 2 "Capacitor_SMD:C_0603_1608Metric_Pad1.05x0.95mm_HandSolder" H 3788 1100 50  0001 C CNN
 F 3 "" H 3750 1250 50  0001 C CNN
 	1    3750 1250
@@
 F 0 "C3" H 4365 1296 50  0000 L CNN
 F 1 "120nF" H 4365 1205 50  0000 L CNN
-F 2 "" H 4288 1100 50  0001 C CNN
+F 2 "Capacitor_SMD:C_0603_1608Metric_Pad1.05x0.95mm_HandSolder" H 4288 1100 50  0001 C CNN
 F 3 "" H 4250 1250 50  0001 C CNN
 	1    4250 1250
@@
 F 0 "R3" H 1330 1296 50  0000 R CNN
 F 1 "10k" H 1330 1205 50  0000 R CNN
-F 2 "" V 1330 1250 50  0001 C CNN
+F 2 "Resistor_SMD:R_0603_1608Metric_Pad1.05x0.95mm_HandSolder" V 1330 1250 50  0001 C CNN
 F 3 "" H 1400 1250 50  0001 C CNN
 	1    1400 1250
@@
 F 0 "R2" H 1080 1296 50  0000 R CNN
 F 1 "10k" H 1080 1205 50  0000 R CNN
-F 2 "" V 1080 1250 50  0001 C CNN
+F 2 "Resistor_SMD:R_0603_1608Metric_Pad1.05x0.95mm_HandSolder" V 1080 1250 50  0001 C CNN
 F 3 "" H 1150 1250 50  0001 C CNN
 	1    1150 1250
@@
 F 0 "R1" H 830 1296 50  0000 R CNN
 F 1 "10k" H 830 1205 50  0000 R CNN
-F 2 "" V 830 1250 50  0001 C CNN
+F 2 "Resistor_SMD:R_0603_1608Metric_Pad1.05x0.95mm_HandSolder" V 830 1250 50  0001 C CNN
 F 3 "" H 900 1250 50  0001 C CNN
 	1    900  1250
@@
 F 0 "R4" H 2030 1296 50  0000 R CNN
 F 1 "10k" H 2030 1205 50  0000 R CNN
-F 2 "" V 2030 1250 50  0001 C CNN
+F 2 "Resistor_SMD:R_0603_1608Metric_Pad1.05x0.95mm_HandSolder" V 2030 1250 50  0001 C CNN
 F 3 "" H 2100 1250 50  0001 C CNN
 	1    2100 1250
@@
 	4950 4150 5600 4150
 Connection ~ 5600 4150
-Wire Wire Line
-	3650 3800 3650 4000
-Connection ~ 3650 4000
-Wire Wire Line
-	3650 4000 3900 4000
 $Comp
 L Connector_Generic:Conn_02x20_Odd_Even J1
@@
 F 0 "J1" H 5500 2917 50  0000 C CNN
 F 1 "JETSON_TX2_CONN" H 5500 2826 50  0000 C CNN
-F 2 "" H 5450 1800 50  0001 C CNN
+F 2 "Connector_PinHeader_2.54mm:PinHeader_2x20_P2.54mm_Vertical" H 5450 1800 50  0001 C CNN
 F 3 "" H 5450 1800 50  0001 C CNN
 	1    5450 1800
@@
 Wire Wire Line
 	1650 3900 1850 3900
-Text Label 3400 3800 0    50   ~ 0
+Text Label 2750 3900 0    50   ~ 0
 MCLR
 Wire Wire Line
-	3400 3800 3650 3800
+	2750 3900 3000 3900
 Text GLabel 5250 3700 0    50   Input ~ 0
 +5V
@@
 F 0 "J3" H 1320 5117 50  0000 C CNN
 F 1 "SERVO1" H 1320 5026 50  0000 C CNN
-F 2 "" H 1400 4800 50  0001 C CNN
+F 2 "Connector_PinHeader_2.54mm:PinHeader_1x03_P2.54mm_Vertical" H 1400 4800 50  0001 C CNN
 F 3 "~" H 1400 4800 50  0001 C CNN
 	1    1400 4800
@@
 F 0 "J4" H 1970 5117 50  0000 C CNN
 F 1 "SERVO2" H 1970 5026 50  0000 C CNN
-F 2 "" H 2050 4800 50  0001 C CNN
+F 2 "Connector_PinHeader_2.54mm:PinHeader_1x03_P2.54mm_Vertical" H 2050 4800 50  0001 C CNN
 F 3 "~" H 2050 4800 50  0001 C CNN
 	1    2050 4800
@@
 F 0 "J5" H 2570 5117 50  0000 C CNN
 F 1 "SERVO3" H 2570 5026 50  0000 C CNN
-F 2 "" H 2650 4800 50  0001 C CNN
+F 2 "Connector_PinHeader_2.54mm:PinHeader_1x03_P2.54mm_Vertical" H 2650 4800 50  0001 C CNN
 F 3 "~" H 2650 4800 50  0001 C CNN
 	1    2650 4800
@@
 Text GLabel 2850 4800 2    50   Input ~ 0
 +12V
+Wire Wire Line
+	3350 4000 3900 4000
+Connection ~ 3000 3900
+Wire Wire Line
+	3000 3900 3000 3800
 $EndSCHEMATC
