File: projects/boat/boat.sch (KiCad schematic (older format))
At the start: 21 parts, among them J10 SERVO2, J11 SERVO3, J12 JETSON_TX2_CONN, J8 SERVO1, J9 PICKIT_CONN, SW0 PIC_RESET, U1 IMU(BNO055), U2 PIC24FV32KA301

Commit message: Combine into hierarchal schematic
Parts:
- removed C28, C30: 100nF, Capacitor_SMD:C_0603_1608Metric_Pad1.05x0.95mm_HandSolder, symbol OARS:C
- removed C29, C34: 100 nF, Capacitor_SMD:C_0603_1608Metric_Pad1.05x0.95mm_HandSolder, symbol OARS:C
- removed C31: 6.8nF, Capacitor_SMD:C_0603_1608Metric_Pad1.05x0.95mm_HandSolder, symbol OARS:C
- removed C32: 120nF, Capacitor_SMD:C_0603_1608Metric_Pad1.05x0.95mm_HandSolder, symbol OARS:C
- removed C33: 10 uF, Capacitor_SMD:C_0603_1608Metric_Pad1.05x0.95mm_HandSolder, symbol OARS:C
- removed J10: SERVO2, Connector_PinHeader_2.54mm:PinHeader_1x03_P2.54mm_Vertical, symbol Connector_Generic:Conn_01x03
- removed J11: SERVO3, Connector_PinHeader_2.54mm:PinHeader_1x03_P2.54mm_Vertical, symbol Connector_Generic:Conn_01x03
- removed J12: JETSON_TX2_CONN, Connector_PinHeader_2.54mm:PinHeader_2x20_P2.54mm_Vertical, symbol Connector_Generic:Conn_02x20_Odd_Even
- removed J8: SERVO1, Connector_PinHeader_2.54mm:PinHeader_1x03_P2.54mm_Vertical, symbol Connector_Generic:Conn_01x03
- removed J9: PICKIT_CONN, Connector_PinHeader_2.54mm:PinHeader_1x05_P2.54mm_Horizontal, symbol Connector_Generic:Conn_01x05
- removed R11, R12, R13, R14, R15: 10k, Resistor_SMD:R_0603_1608Metric_Pad1.05x0.95mm_HandSolder, symbol Device:R
- removed R16: 470, Resistor_SMD:R_0603_1608Metric_Pad1.05x0.95mm_HandSolder, symbol Device:R
- removed SW0: PIC_RESET, symbol Switch:SW_Push
- removed U1: IMU(BNO055), Package_LGA:LGA-28_5.2x3.8mm_P0.5mm, symbol Sensor_Motion:BNO055
- removed U2: PIC24FV32KA301, OARS:PIC24FV32KA301-SOIC, symbol OARS:PIC24FV32KA301
Connections:
- net labels removed: GND, MCLR, M_INT, OC1, OC2, OC3, PGEC, PGED, SCK1, SCL, SDA, SDI1, SDO1, SS1, VDD12, VDD3.3, VDD5
- wire segments 69 -> 0
Other:
- note removed: "1: MCLR, Master Clear\n2: PGEC, Programmer Communication \n3: PGED, Programmer Communication \n4: OC2, PWM for servo #2\n5: OC3, PWM for servo #3\n11: OC1, PWM for servo #1\n14: VCAP, see PIC datasheet\n15: SCK1, SPI Clock\n16: SDO1, SPI Data Out\n17: SDI1, SPI Data In\n18: SS1, Slave Select1 (input)\n19: VSS, Ground\n20: VDD, VDD5 Supply"
- note removed: "Designer: Michael Remley"
- note removed: "IMU (Motion Sensor)\nConnected directly to Jetson\nI2C Addr.: 0x28"
- note removed: "PICKIT3 Connector\nfor Programming"
- note removed: "SPI Connection:\nPIC operates as Slave\nSDI1 is Master Out/Slave In\nSDO1 is Master In/Slave out\nSS1 is Active-Low Slave Select"
- note removed: "Servo Control Connector\nSignals and 12V Power\nOC1, OC2, & OC3 are 5V PWM"
- note removed: "uController"
