File: projects/power_adapter/power_adapter.sch (KiCad schematic (older format))
At the start: 49 parts, among them J0 USB3_A, J1 USB3_A, J2 USB3_A, J3 USB3_A, J4 USB3_A, J5 USB_A, J6 USB_A, J7 USB_A, U0 USB5537B, Y0 XTAL_GND

Commit message: Add power adapter
Update USB hub and misc assets
Parts:
- removed C0, C10, C13, C15, C16, C17, C2, C4, C6, C8: 0.1uF, symbol OARS:C
- removed C18, C19: 6pF, symbol OARS:C
- removed C20: 1nF, symbol OARS:C
- removed C21, C22, C23, C24, C25, C26, C27: 150uF, symbol Device:CP1
- removed J0, J1, J2, J3, J4: USB3_A, symbol OARS:USB3_A
- removed J5, J6, J7: USB_A, symbol OARS:USB_A
- removed U0: USB5537B, symbol OARS:USB5537B
- removed Y0: XTAL_GND, symbol OARS:XTAL_GND
- added C0, C12, C4, C8: 100uF, symbol Device:CP1
- added C10, C13, C2, C6: 470uF, symbol Device:CP1
- added D0, D1, D2, D3: D_Zener, symbol Device:D_Zener
- added L0, L2, L4, L6: 220uH, symbol Device:L_Core_Iron
- added L1, L3, L5, L7: 1uH, symbol Device:L_Core_Iron
- added R11: 30k, symbol OARS:R
- added U0, U1, U2, U3: AZ34063U, symbol OARS:AZ34063U
- C1, C12, C5, C9: value 0.1uF -> 470pF
- C11, C14, C3, C7: value 0.1uF -> 100uF
- R0, R3, R6: value 330 -> 0.33
- R1: value 330 -> 10k
- R10: value 12k -> 1.2k
- R2, R5: value 330 -> 1.2k
- R4: value 330 -> 3.6k
- R7: value 330 -> 2k
- R8: value 100k -> 1.2k
- R9: value 100k -> 0.33
Connections:
- net labels added: VCC, VDD12, VDD5
- net labels removed: 5V_PRT1, 5V_PRT2, 5V_PRT3, 5V_PRT4, 5V_PRT5, 5V_PRT6, 5V_PRT7, PRTSHD_1, PRTSHD_2, PRTSHD_3, PRTSHD_4, PRTSHD_5, PRTSHD_6, PRTSHD_7, PRTSHD_UP, VBUS
- wire segments 252 -> 78
- no-connect marks 13 -> 0

Commit message: Combine into hierarchal schematic
Parts:
- renumbered C8 to C35, C0 to C36, C9 to C37, C1 to C38, C10 to C39, C2 to C40, C11 to C41, C3 to C42, C12 to C43, C4 to C44, C12 to C45, C5 to C46, C13 to C47, C6 to C48, C14 to C49, C7 to C50, D2 to D0, D0 to D1, D3 to D2, D1 to D3, L4 to L0, L0 to L1, L5 to L2, L1 to L3, L6 to L4, L2 to L5, L7 to L6, L3 to L7, R6 to R17, R0 to R18, R8 to R19, R2 to R20, R7 to R21, R1 to R22, R9 to R23, R3 to R24, R11 to R25, R5 to R26, R10 to R27, R4 to R28, U2 to U3, U0 to U4, U3 to U5, U1 to U6
Connections:
- wire segments 78 -> 80

Commit message: Reorganize and add full boat schematic
For the future, let's not delete old documentation files. Just add a new one and update the date. It''ll be useful for our decision process and for others who would like to track our progress
Parts:
- U3, U4, U5, U6: footprint (none) -> Package_SO:SOIC-8_3.9x4.9mm_P1.27mm
Changed lines of the file:
@@
 EESchema Schematic File Version 4
-LIBS:power_adapter-cache
-LIBS:uController_hub-cache
+LIBS:boat-cache
 EELAYER 26 0
 EELAYER END
@@
 F 0 "U4" H 1600 3350 50  0000 C CNN
 F 1 "AZ34063U" H 2000 3350 50  0000 C CNN
-F 2 "" H 2000 3200 50  0001 C CNN
+F 2 "Package_SO:SOIC-8_3.9x4.9mm_P1.27mm" H 2000 3200 50  0001 C CNN
 F 3 "" H 2000 3200 50  0001 C CNN
 	1    2000 3100
@@
 F 0 "U6" H 4450 3350 50  0000 C CNN
 F 1 "AZ34063U" H 4850 3350 50  0000 C CNN
-F 2 "" H 4850 3200 50  0001 C CNN
+F 2 "Package_SO:SOIC-8_3.9x4.9mm_P1.27mm" H 4850 3200 50  0001 C CNN
 F 3 "" H 4850 3200 50  0001 C CNN
 	1    4850 3100
@@
 F 0 "U3" H 1600 1400 50  0000 C CNN
 F 1 "AZ34063U" H 2000 1400 50  0000 C CNN
-F 2 "" H 2000 1250 50  0001 C CNN
+F 2 "Package_SO:SOIC-8_3.9x4.9mm_P1.27mm" H 2000 1250 50  0001 C CNN
 F 3 "" H 2000 1250 50  0001 C CNN
 	1    2000 1150
@@
 F 0 "U5" H 4450 1400 50  0000 C CNN
 F 1 "AZ34063U" H 4850 1400 50  0000 C CNN
-F 2 "" H 4850 1250 50  0001 C CNN
+F 2 "Package_SO:SOIC-8_3.9x4.9mm_P1.27mm" H 4850 1250 50  0001 C CNN
 F 3 "" H 4850 1250 50  0001 C CNN
 	1    4850 1150
