File: projects/usb/usb.sch (KiCad schematic (older format))
At the start: 71 parts, among them J0 USB3_A, J1 USB3_A, J2 USB3_A, J3 USB3_A, J4 USB3_A, J5 USB_A, J6 USB_A, J7 USB_A, U0 USB5537B, U1 AZ34063U, U2 AZ34063U, Y0 XTAL_GND

Commit message: Add power adapter
Update USB hub and misc assets
Parts:
- removed C28, C32: 100uF, symbol Device:CP1
- removed C29, C33: 470pF, symbol OARS:C
- removed C30, C34: 470uF, symbol Device:CP1
- removed C31, C35: 100uF, symbol OARS:C
- removed D0, D1: D_Zener, symbol Device:D_Zener
- removed L0, L2: 220uH, symbol Device:L_Core_Iron
- removed L1, L3: 1uH, symbol Device:L_Core_Iron
- removed R11, R14: 0.33, symbol OARS:R
- removed R12: 2k, symbol OARS:R
- removed R13, R16: 1.2k, symbol OARS:R
- removed R15: 100k, symbol OARS:R
- removed U1, U2: AZ34063U, symbol OARS:AZ34063U
Connections:
- net labels added: VDD1.2, VDD3.3
- net labels removed: VCC, VDD12, VDD33
- wire segments 291 -> 252

Commit message: Combine into hierarchal schematic
Parts:
- renumbered C25 to C0, C20 to C1, C14 to C10, C23 to C11, C18 to C12, C19 to C13, C13 to C14, C11 to C15, C12 to C16, C10 to C17, C22 to C18, C21 to C19, C26 to C2, C0 to C20, C2 to C21, C4 to C22, C6 to C23, C1 to C24, C3 to C25, C5 to C26, C7 to C27, C27 to C3, C16 to C4, C24 to C5, C17 to C6, C8 to C7, C9 to C8, C15 to C9, J5 to J0, J6 to J1, J4 to J2, J7 to J3, J3 to J4, J0 to J5, J2 to J6, J1 to J7, R8 to R0, R9 to R1, R7 to R10, R10 to R2, R0 to R3, R2 to R4, R4 to R5, R1 to R7, R3 to R8, R5 to R9
Connections:
- wire segments 252 -> 255

Commit message: Reorganize and add full boat schematic
For the future, let's not delete old documentation files. Just add a new one and update the date. It''ll be useful for our decision process and for others who would like to track our progress
Parts:
- C0, C1, C10, C11, C12, C13, C14, C15, C16, C17, C18, C19, C2, C20, C21, C22, C23, C24, C25, C26, C27, C3, C4, C5, C6, C7, C8, C9: footprint (none) -> Capacitor_SMD:C_0603_1608Metric_Pad1.05x0.95mm_HandSolder
- J0, J1, J3: footprint (none) -> Connector_USB:USB_A_CNCTech_1001-011-01101_Horizontal
- J2, J4, J5, J6, J7: footprint (none) -> Connector_USB:USB3_A_Molex_48393-001
- R0, R1, R10, R2, R3, R4, R5, R6, R7, R8, R9: footprint (none) -> Resistor_SMD:R_0603_1608Metric_Pad1.05x0.95mm_HandSolder
- U0: footprint (none) -> OARS:Microchip_USB5537B_QFN-72
- Y0: value XTAL_GND -> 25M_XTAL
